Commit message: initial commit

File: src/allegro_hand_description/fixed_urdf.urdf (robot description, URDF)
Before this commit: robot allegro_hand_left, 21 links, 20 joints
Links:
- added link dummy
- link link_12.0: geometry collision box size=0.0358 0.034 0.0455; visual mesh filename=package://allegro_hand_description/meshes/link_12.0_right.S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
- link palm_link: geometry collision box size=0.0408 0.1130 0.095; visual mesh filename=package://allegro_hand_description/meshes/base_link.STL
Joints:
- added joint dummy_joint: type fixed, parent dummy, child palm_link
- joint joint_0.0: origin xyz=0 -0.0435 -0.001542 rpy=0.08726646255 0 0 -> xyz=0 0.0435 -0.001542 rpy=-0.08726646255 0 0
- joint joint_12.0: axis +1 0 0 -> -1 0 0; origin xyz=-0.0182 -0.019333 -0.045987 rpy=0 -1.65806278845 1.5707963259 -> xyz=-0.0182 0.019333 -0.045987 rpy=0 -1.65806278845 -1.5707963259
- joint joint_13.0: axis 0 0 -1 -> 0 0 1; origin xyz=-0.027 -0.005 0.0399 -> xyz=-0.027 0.005 0.0399
- joint joint_8.0: origin xyz=0 0.0435 -0.001542 rpy=-0.08726646255 0 0 -> xyz=0 -0.0435 -0.001542 rpy=0.08726646255 0 0
